Commit message: Booster K1 full integration and mesh fixes
- Updated K1 URDF mesh paths to match actual asset locations, resolving all visual/collision errors in Isaac Gym
- Verified and fixed buffer/loop logic for multi-robot support
- Ensured K1 robot loads and runs successfully in simulation (minimal_k1_example.py)
- Improved minimal example to keep viewer open for presentations

File: resources/robots/k1/urdf/k1.urdf (robot description, URDF)
Before this commit: robot K1, 25 links, 24 joints
Links:
- link Head_1: geometry collision mesh filename=resources/robots/k1/meshes/Head_1.STL; visual mesh filename=resources/robots/k1/meshes/Head_1.STL
- link Head_2: geometry collision mesh filename=resources/robots/k1/meshes/Head_2.STL; visual mesh filename=resources/robots/k1/meshes/Head_2.STL
- link Left_Ankle_Cross: geometry visual mesh filename=resources/robots/k1/meshes/Left_Ankle_Cross.STL
- link Left_Arm_1: geometry visual mesh filename=resources/robots/k1/meshes/Left_Arm_1.STL
- link Left_Arm_2: geometry collision cylinder length=0.068 radius=0.035; visual mesh filename=resources/robots/k1/meshes/Left_Arm_2.STL
- link Left_Arm_3: geometry collision mesh filename=resources/robots/k1/meshes/Left_Arm_3.STL; visual mesh filename=resources/robots/k1/meshes/Left_Arm_3.STL
- link Left_Hip_Pitch: geometry visual mesh filename=resources/robots/k1/meshes/Left_Hip_Pitch.STL
- link Left_Hip_Roll: geometry collision cylinder length=0.094 radius=0.036; visual mesh filename=resources/robots/k1/meshes/Left_Hip_Roll.STL
- link Left_Hip_Yaw: geometry collision cylinder length=0.066 radius=0.04; visual mesh filename=resources/robots/k1/meshes/Left_Hip_Yaw.STL
- link Left_Shank: geometry collision box size=0.06 0.06 0.10; collision cylinder length=0.07 radius=0.045
- link Right_Ankle_Cross: geometry visual mesh filename=resources/robots/k1/meshes/Right_Ankle_Cross.STL
- link Right_Arm_1: geometry visual mesh filename=resources/robots/k1/meshes/Right_Arm_1.STL
- link Right_Arm_2: geometry collision cylinder length=0.068 radius=0.035; visual mesh filename=resources/robots/k1/meshes/Right_Arm_2.STL
- link Right_Arm_3: geometry collision mesh filename=resources/robots/k1/meshes/Right_Arm_3.STL; visual mesh filename=resources/robots/k1/meshes/Right_Arm_3.STL
- link Right_Hip_Pitch: geometry visual mesh filename=resources/robots/k1/meshes/Right_Hip_Pitch.STL
- link Right_Hip_Roll: geometry collision cylinder length=0.094 radius=0.036; visual mesh filename=resources/robots/k1/meshes/Right_Hip_Roll.STL
- link Right_Hip_Yaw: geometry collision cylinder length=0.066 radius=0.04; visual mesh filename=resources/robots/k1/meshes/Right_Hip_Yaw.STL
- link Right_Shank: geometry collision box size=0.06 0.06 0.1; collision cylinder length=0.07 radius=0.045
- link Trunk: geometry collision box size=0.12 0.18 0.2; collision cylinder length=0.1 radius=0.05
- link left_foot_link: geometry collision mesh filename=resources/robots/k1/meshes/Left_Foot.STL; visual mesh filename=resources/robots/k1/meshes/Left_Foot.STL
- link left_hand_link: geometry collision mesh filename=resources/robots/k1/meshes/Left_Arm_4.STL; visual mesh filename=resources/robots/k1/meshes/Left_Arm_4.STL
- link right_foot_link: geometry collision mesh filename=resources/robots/k1/meshes/Right_Foot.STL; visual mesh filename=resources/robots/k1/meshes/Right_Foot.STL
- link right_hand_link: geometry collision mesh filename=resources/robots/k1/meshes/Right_Arm_4.STL; visual mesh filename=resources/robots/k1/meshes/Right_Arm_4.STL
